File: pcb-design/HiveScale_V0.kicad_sch (KiCad schematic)
At the start: 25 parts, among them J1 ESP32-left-RXTX, J10 PowerIn, J11 Loadcell1-Input, J12 Loadcell2-Input, J13 DS18B20 Hive1, J14 DS18B20 Hive2, J15 SHT40 Ambient, J16 SolarPowerIn and INA219, J17 CN3971, J18 TPS63020-GND-OUT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

Commit message: Waeninf and Iteration
Connections:
- net +5V: now also J20.1 (Pin_1)
- net 3.3V: no longer J20.1 (Pin_1)
Changed lines of the file:
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@@
 	)
 	(junction
+		(at 55.88 43.18)
+		(diameter 0)
+		(color 0 0 0 0)
+	)
+	(junction
 		(at 148.59 119.38)
 		(diameter 0)
@@
 	)
 	(junction
-		(at 53.34 143.51)
-		(diameter 0)
-		(color 0 0 0 0)
-	)
-	(junction
 		(at 85.09 35.56)
 		(diameter 0)
@@
 	(wire
 		(pts
+			(xy 55.88 43.18) (xy 55.88 116.84)
+		)
+		(stroke
+			(width 0)
+			(type default)
+		)
+	)
+	(wire
+		(pts
 			(xy 127 83.82) (xy 127 88.9)
 		)
@@
 	(wire
 		(pts
-			(xy 26.67 116.84) (xy 53.34 116.84)
+			(xy 26.67 116.84) (xy 55.88 116.84)
 		)
 		(stroke
@@
 	(wire
 		(pts
-			(xy 34.29 43.18) (xy 64.77 43.18)
+			(xy 34.29 43.18) (xy 55.88 43.18)
 		)
 		(stroke
@@
 	(wire
 		(pts
-			(xy 53.34 116.84) (xy 53.34 143.51)
+			(xy 209.55 120.65) (xy 209.55 119.38)
 		)
 		(stroke
@@
 	(wire
 		(pts
-			(xy 209.55 120.65) (xy 209.55 119.38)
+			(xy 118.11 72.39) (xy 118.11 81.28)
 		)
 		(stroke
@@
 	(wire
 		(pts
-			(xy 118.11 72.39) (xy 118.11 81.28)
+			(xy 49.53 146.05) (xy 49.53 170.18)
 		)
 		(stroke
@@
 	(wire
 		(pts
-			(xy 49.53 146.05) (xy 49.53 170.18)
+			(xy 160.02 83.82) (xy 158.75 83.82)
 		)
 		(stroke
@@
 	(wire
 		(pts
-			(xy 160.02 83.82) (xy 158.75 83.82)
+			(xy 229.87 52.07) (xy 210.82 52.07)
 		)
 		(stroke
@@
 	(wire
 		(pts
-			(xy 229.87 52.07) (xy 210.82 52.07)
+			(xy 212.09 60.96) (xy 199.39 60.96)
 		)
 		(stroke
@@
 	(wire
 		(pts
-			(xy 212.09 60.96) (xy 199.39 60.96)
+			(xy 229.87 73.66) (xy 229.87 76.2)
 		)
 		(stroke
@@
 	(wire
 		(pts
-			(xy 229.87 73.66) (xy 229.87 76.2)
+			(xy 55.88 43.18) (xy 64.77 43.18)
 		)
 		(stroke
@@
 					(size 1.27 1.27)
 				)
-				(justify left)
+				(justify right)
 			)
 		)
@@
 		)
 		(property "Value" "TPS63020-3.3V-OUT"
-			(at 74.93 35.5599 0)
+			(at 77.216 33.02 0)
 			(effects
 				(font
 					(size 1.27 1.27)
 				)
-				(justify left)
+				(justify right)
 			)
 		)
