File: pcb-design/power module/_V0_3-Power_Module.kicad_pcb (KiCad board)
At the start: 2 copper layers, 76 x 56 mm, 17 parts, among them J16 SolarPowerIn and INA219, J17 CN3971, J18 TPS63020-GND-OUT, J19 TPS63020-V-IN, J20 ConnectorHiveScale, J21 MAXS17048, J23 TPS63020-3.3V-OUT, J6 TPS63020-GND-IN, m3-bl MountingHole_3.2mm_M3, m3-br MountingHole_3.2mm_M3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

Commit message: updated v0.3 pcb design
Connections:
- J16 pad 5: /BATneg -> /Solarpos
- J16 pad 6: /Solarpos -> unconnected-(J16-Pin_6-Pad6)
Routing:
- net /Solarpos: track 41.3 -> 40.2 mm
- net /BATneg: vias 51 -> 52
Changed lines of the file:
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@@
 		(property ki_fp_filters "Connector*:*_1x??_*")
 		(sheetname "/")
-		(sheetfile "_V0_2-Power_Module.kicad_sch")
+		(sheetfile "_V0_3-Power_Module.kicad_sch")
+		(units
+			(unit
+				(name "A")
+				(pins "1" "2")
+			)
+		)
 		(attr through_hole)
 		(duplicate_pad_numbers_are_jumpers no)
@@
 		(property ki_fp_filters "Connector*:*_1x??_*")
 		(sheetname "/")
-		(sheetfile "_V0_2-Power_Module.kicad_sch")
+		(sheetfile "_V0_3-Power_Module.kicad_sch")
+		(units
+			(unit
+				(name "A")
+				(pins "1" "2")
+			)
+		)
 		(attr through_hole)
 		(duplicate_pad_numbers_are_jumpers no)
@@
 		(property ki_fp_filters "Connector*:*_1x??_*")
 		(sheetname "/")
-		(sheetfile "_V0_2-Power_Module.kicad_sch")
+		(sheetfile "_V0_3-Power_Module.kicad_sch")
+		(units
+			(unit
+				(name "A")
+				(pins "1" "2" "3" "4" "5" "6")
+			)
+		)
 		(attr through_hole)
 		(duplicate_pad_numbers_are_jumpers no)
@@
 			(layers "*.Cu" "*.Mask")
 			(remove_unused_layers no)
-			(net "/BATneg")
+			(net "/Solarpos")
 			(pinfunction "Pin_5_5")
 			(pintype "passive")
@@
 			(layers "*.Cu" "*.Mask")
 			(remove_unused_layers no)
-			(net "/Solarpos")
+			(net "unconnected-(J16-Pin_6-Pad6)")
 			(pinfunction "Pin_6_6")
 			(pintype "passive")
@@
 		(property ki_fp_filters "Connector*:*_1x??_*")
 		(sheetname "/")
-		(sheetfile "_V0_2-Power_Module.kicad_sch")
+		(sheetfile "_V0_3-Power_Module.kicad_sch")
+		(units
+			(unit
+				(name "A")
+				(pins "1" "2" "3" "4" "5" "6")
+			)
+		)
 		(attr through_hole)
 		(duplicate_pad_numbers_are_jumpers no)
@@
 		(property ki_fp_filters "Connector*:*_1x??_*")
 		(sheetname "/")
-		(sheetfile "_V0_2-Power_Module.kicad_sch")
+		(sheetfile "_V0_3-Power_Module.kicad_sch")
+		(units
+			(unit
+				(name "A")
+				(pins "1" "2")
+			)
+		)
 		(attr through_hole)
 		(duplicate_pad_numbers_are_jumpers no)
@@
 		(property ki_fp_filters "Connector*:*_1x??_*")
 		(sheetname "/")
-		(sheetfile "_V0_2-Power_Module.kicad_sch")
+		(sheetfile "_V0_3-Power_Module.kicad_sch")
+		(units
+			(unit
+				(name "A")
+				(pins "1" "2")
+			)
+		)
 		(attr through_hole)
 		(duplicate_pad_numbers_are_jumpers no)
@@
 		(property ki_fp_filters "Connector*:*_1x??_*")
 		(sheetname "/")
-		(sheetfile "_V0_2-Power_Module.kicad_sch")
+		(sheetfile "_V0_3-Power_Module.kicad_sch")
+		(units
+			(unit
+				(name "A")
+				(pins "1" "2" "3" "4" "5" "6")
+			)
+		)
 		(attr through_hole)
 		(duplicate_pad_numbers_are_jumpers no)
@@
 		(property ki_fp_filters "Connector*:*_1x??_*")
 		(sheetname "/")
-		(sheetfile "_V0_2-Power_Module.kicad_sch")
+		(sheetfile "_V0_3-Power_Module.kicad_sch")
+		(units
+			(unit
+				(name "A")
+				(pins "1" "2")
+			)
+		)
 		(attr through_hole)
 		(duplicate_pad_numbers_are_jumpers no)
@@
 		(property ki_fp_filters "Connector*:*_1x??_*")
 		(sheetname "/")
-		(sheetfile "_V0_2-Power_Module.kicad_sch")
+		(sheetfile "_V0_3-Power_Module.kicad_sch")
+		(units
+			(unit
+				(name "A")
+				(pins "1" "2" "3" "4")
+			)
+		)
 		(attr through_hole)
 		(duplicate_pad_numbers_are_jumpers no)
@@
 		(property ki_fp_filters "Connector*:*_1x??_*")
 		(sheetname "/")
-		(sheetfile "_V0_2-Power_Module.kicad_sch")
+		(sheetfile "_V0_3-Power_Module.kicad_sch")
+		(units
+			(unit
+				(name "A")
+				(pins "1" "2")
+			)
+		)
 		(attr through_hole)
 		(duplicate_pad_numbers_are_jumpers no)
@@
 		(property ki_fp_filters "Connector*:*_1x??_*")
 		(sheetname "/")
-		(sheetfile "_V0_2-Power_Module.kicad_sch")
+		(sheetfile "_V0_3-Power_Module.kicad_sch")
+		(units
+			(unit
+				(name "A")
+				(pins "1" "2")
+			)
+		)
 		(attr through_hole)
 		(duplicate_pad_numbers_are_jumpers no)
@@
 	)
 	(via
-		(at 159.5 64)
+		(at 158.5 64.5)
 		(size 0.6)
 		(drill 0.4)
@@
 	)
 	(via
+		(at 154.5 60)
+		(size 0.6)
+		(drill 0.4)
+		(layers "F.Cu" "B.Cu")
+		(free yes)
+		(net "/BATneg")
+	)
+	(via
 		(at 159 79.5)
 		(size 0.6)
@@
 	)
 	(segment
-		(start 154.1998 69.8701)
-		(end 157.043 69.8701)
+		(start 161.835 65.0781)
+		(end 161.835 62)
 		(width 2)
 		(layer "B.Cu")
@@
 	)
 	(segment
-		(start 135.12 88.9499)
-		(end 154.1998 69.8701)
+		(start 154.1998 69.8701)
+		(end 157.043 69.8701)
 		(width 2)
 		(layer "B.Cu")
@@
 	)
 	(segment
-		(start 164.375 62.5381)
-		(end 164.375 62)
+		(start 157.043 69.8701)
+		(end 161.835 65.0781)
 		(width 2)
 		(layer "B.Cu")
@@
 	)
 	(segment
-		(start 135.12 89.475)
-		(end 135.12 88.9499)
+		(start 135.12 88.9499)
+		(end 154.1998 69.8701)
 		(width 2)
 		(layer "B.Cu")
@@
 	)
 	(segment
-		(start 157.043 69.8701)
-		(end 164.375 62.5381)
+		(start 135.12 89.475)
+		(end 135.12 88.9499)
 		(width 2)
 		(layer "B.Cu")
@@
 		(members "4d1eee34-cdf9-4274-9a69-0f9461c4f1b4" "4ef4a140-7314-49bf-89d2-7c22268e71af"
 			"5dc73560-5788-4075-a74a-bd636093a09b" "5ff5eb13-dab4-4deb-98a4-c377d7dea667"
-			"734fd407-b7dd-4883-b677-620da57d70ab" "839efebb-4932-458b-8b15-d1ffa648c10e"
-			"933361c1-72ae-4e2c-871d-5b45fad0a2fa" "a6fcb528-e400-49f9-a5db-28d980f85b8b"
-			"e92c0f76-8ba1-4046-875f-0a1c006d827c"
+			"734fd407-b7dd-4883-b677-620da57d70ab" "933361c1-72ae-4e2c-871d-5b45fad0a2fa"
+			"a6fcb528-e400-49f9-a5db-28d980f85b8b" "e92c0f76-8ba1-4046-875f-0a1c006d827c"
 		)
 	)
 	(group ""
+		(members "4115d001-d9d1-488b-8464-f7c317f6ec78" "be1261ae-86e3-4509-a3c9-527d2b40b858")
+	)
+	(group ""
 		(members "4e26c16a-8dc7-4396-a722-daca5e8765b5" "63760b51-b387-4ce0-b7f3-4b1c982805ec"
 			"7b08cfab-526c-4a4c-816e-753539e61198" "cc81f62b-b49a-4a90-a19d-8a48c42c66c0"
-			"dcfaf176-12e6-4fc1-822c-5c810059fa5d" "e74bb63e-ac60-4414-a03b-5d712516a8be"
+			"dcfaf176-12e6-4fc1-822c-5c810059fa5d"
 		)
 	)
 	(group ""
-		(members "4115d001-d9d1-488b-8464-f7c317f6ec78" "be1261ae-86e3-4509-a3c9-527d2b40b858")
-	)
-	(group ""
