File: pcb-design/power module/_V0_3-Power_Module.kicad_sch (KiCad schematic)
At the start: 11 parts, among them J16 SolarPowerIn and INA219, J17 CN3971, J18 TPS63020-GND-OUT, J19 TPS63020-V-IN, J20 ConnectorHiveScale, J21 MAXS17048, J23 TPS63020-3.3V-OUT, J6 TPS63020-GND-IN

Commit message: updated v0.3 pcb design
Connections:
- net BATneg: no longer J16.5 (Pin_5)
- net Solarpos: now also J16.5 (Pin_5); no longer J16.6 (Pin_6)
Changed lines of the file:
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@@
+		)
+	)
+	(label "Solarpos"
+		(at 92.71 54.61 0)
+		(effects
+			(font
+				(size 1.27 1.27)
+			)
+			(justify left bottom)
 		)
 	)
@@
 		)
 	)
-	(label "Solarpos"
-		(at 92.71 57.15 0)
-		(effects
-			(font
-				(size 1.27 1.27)
-			)
-			(justify left bottom)
-		)
-	)
 	(label "GND"
 		(at 198.12 58.42 0)
@@
 	(label "SCL"
 		(at 198.12 68.58 0)
-		(effects
-			(font
-				(size 1.27 1.27)
-			)
-			(justify left bottom)
-		)
-	)
-	(label "Solarneg"
-		(at 92.71 54.61 0)
 		(effects
 			(font
@@
 		)
 		(instances
-			(project "_V0_2-Power_Module"
+			(project "_V0_3-Power_Module"
 				(path "/0fd72f3f-0d89-4c92-9f9e-d7a48828e0f6"
 					(reference "J21")
@@
 		)
 		(instances
-			(project "_V0_2-Power_Module"
+			(project "_V0_3-Power_Module"
 				(path "/0fd72f3f-0d89-4c92-9f9e-d7a48828e0f6"
 					(reference "TP4056-1")
@@
 		)
 		(instances
-			(project "_V0_2-Power_Module"
+			(project "_V0_3-Power_Module"
 				(path "/0fd72f3f-0d89-4c92-9f9e-d7a48828e0f6"
 					(reference "J18")
@@
 		)
 		(instances
-			(project "_V0_2-Power_Module"
+			(project "_V0_3-Power_Module"
 				(path "/0fd72f3f-0d89-4c92-9f9e-d7a48828e0f6"
 					(reference "J16")
@@
 		)
 		(instances
-			(project "_V0_2-Power_Module"
+			(project "_V0_3-Power_Module"
 				(path "/0fd72f3f-0d89-4c92-9f9e-d7a48828e0f6"
 					(reference "J19")
@@
 		)
 		(instances
-			(project "_V0_2-Power_Module"
+			(project "_V0_3-Power_Module"
 				(path "/0fd72f3f-0d89-4c92-9f9e-d7a48828e0f6"
 					(reference "MAX17048")
@@
 		)
 		(instances
-			(project "_V0_2-Power_Module"
+			(project "_V0_3-Power_Module"
 				(path "/0fd72f3f-0d89-4c92-9f9e-d7a48828e0f6"
 					(reference "J20")
@@
 		)
 		(instances
-			(project "_V0_2-Power_Module"
+			(project "_V0_3-Power_Module"
 				(path "/0fd72f3f-0d89-4c92-9f9e-d7a48828e0f6"
 					(reference "J6")
@@
 		)
 		(instances
-			(project "_V0_2-Power_Module"
+			(project "_V0_3-Power_Module"
 				(path "/0fd72f3f-0d89-4c92-9f9e-d7a48828e0f6"
 					(reference "TP4056+1")
@@
 		)
 		(instances
-			(project "_V0_2-Power_Module"
+			(project "_V0_3-Power_Module"
 				(path "/0fd72f3f-0d89-4c92-9f9e-d7a48828e0f6"
 					(reference "J23")
@@
 		)
 		(instances
-			(project "_V0_2-Power_Module"
+			(project "_V0_3-Power_Module"
 				(path "/0fd72f3f-0d89-4c92-9f9e-d7a48828e0f6"
 					(reference "J17")
